File: schematics/pm_sensor/pm_sensor.kicad_pcb (KiCad board)
At the start: 2 copper layers, 71.1 x 30.5 mm, 19 parts, among them J1 sds011_conn, J3 conn_display, Q1 2N7000TA, Q2 2N7000TA, Q3 2N7000TA, Q4 IRF9510, U1 WeMos_D1_mini, U2 DHT22

Commit message: Add pulldown on SDS011 switch pin
Parts:
- added R9: 10k, Resistor_THT:R_Axial_DIN0207_L6.3mm_D2.5mm_P10.16mm_Horizontal, B.Cu at (43.2, 27.9)
Changed lines of the file:
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@@
     (tracks 45)
     (zones 0)
-    (modules 19)
+    (modules 20)
     (nets 25)
   )
@@
     (add_net sds_vcc)
   )
+  (module Resistor_THT:R_Axial_DIN0207_L6.3mm_D2.5mm_P10.16mm_Horizontal (layer B.Cu)
+    (at 43.18 27.94 180)
+    (descr "Resistor, Axial_DIN0207 series, Axial, Horizontal, pin pitch=10.16mm, 0.25W = 1/4W, length*diameter=6.3*2.5mm^2, http://cdn-reichelt.de/documents/datenblatt/B400/1_4W%23YAG.pdf")
+    (tags "Resistor Axial_DIN0207 series Axial Horizontal pin pitch 10.16mm 0.25W = 1/4W length 6.3mm diameter 2.5mm")
+    (fp_text reference R9 (at 5.08 2.37 180) (layer B.SilkS)
+      (effects (font (size 1 1) (thickness 0.15)) (justify mirror))
+    )
+    (fp_text value 10k (at 5.08 -2.37 180) (layer B.Fab)
+      (effects (font (size 1 1) (thickness 0.15)) (justify mirror))
+    )
+    (fp_text user %R (at 5.08 0 180) (layer B.Fab)
+      (effects (font (size 1 1) (thickness 0.15)) (justify mirror))
+    )
+    (fp_line (start 11.21 1.5) (end -1.05 1.5) (layer B.CrtYd) (width 0.05))
+    (fp_line (start 11.21 -1.5) (end 11.21 1.5) (layer B.CrtYd) (width 0.05))
+    (fp_line (start -1.05 -1.5) (end 11.21 -1.5) (layer B.CrtYd) (width 0.05))
+    (fp_line (start -1.05 1.5) (end -1.05 -1.5) (layer B.CrtYd) (width 0.05))
+    (fp_line (start 9.12 0) (end 8.35 0) (layer B.SilkS) (width 0.12))
+    (fp_line (start 1.04 0) (end 1.81 0) (layer B.SilkS) (width 0.12))
+    (fp_line (start 8.35 1.37) (end 1.81 1.37) (layer B.SilkS) (width 0.12))
+    (fp_line (start 8.35 -1.37) (end 8.35 1.37) (layer B.SilkS) (width 0.12))
+    (fp_line (start 1.81 -1.37) (end 8.35 -1.37) (layer B.SilkS) (width 0.12))
+    (fp_line (start 1.81 1.37) (end 1.81 -1.37) (layer B.SilkS) (width 0.12))
+    (fp_line (start 10.16 0) (end 8.23 0) (layer B.Fab) (width 0.1))
+    (fp_line (start 0 0) (end 1.93 0) (layer B.Fab) (width 0.1))
+    (fp_line (start 8.23 1.25) (end 1.93 1.25) (layer B.Fab) (width 0.1))
+    (fp_line (start 8.23 -1.25) (end 8.23 1.25) (layer B.Fab) (width 0.1))
+    (fp_line (start 1.93 -1.25) (end 8.23 -1.25) (layer B.Fab) (width 0.1))
+    (fp_line (start 1.93 1.25) (end 1.93 -1.25) (layer B.Fab) (width 0.1))
+    (pad 2 thru_hole oval (at 10.16 0 180) (size 1.6 1.6) (drill 0.8) (layers *.Cu *.Mask)
+      (net 14 GND))
+    (pad 1 thru_hole circle (at 0 0 180) (size 1.6 1.6) (drill 0.8) (layers *.Cu *.Mask)
+      (net 21 "Net-(Q3-Pad2)"))
+    (model ${KISYS3DMOD}/Resistor_THT.3dshapes/R_Axial_DIN0207_L6.3mm_D2.5mm_P10.16mm_Horizontal.wrl
+      (at (xyz 0 0 0))
+      (scale (xyz 1 1 1))
+      (rotate (xyz 0 0 0))
+    )
+  )
   (module Capacitor_THT:C_Disc_D5.0mm_W2.5mm_P5.00mm (layer F.Cu)

Commit message: Some unknown schematic changes [skip ci]
Parts:
- moved R9 9.16 mm to (38.1, 20.3), turned to 270 degrees
Routing:
- net sds_switch: track 10.2 -> 0.00 mm
- net GND: track 35.4 -> 37.9 mm
- net Net-(Q3-Pad2): track 7.62 -> 10.2 mm
- net +5V: track 53.3 -> 50.8 mm
Changed lines of the file:
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@@
     (thickness 1.6)
     (drawings 12)
-    (tracks 45)
+    (tracks 43)
     (zones 0)
     (modules 20)
@@
   )
   (module Resistor_THT:R_Axial_DIN0207_L6.3mm_D2.5mm_P10.16mm_Horizontal (layer B.Cu)
-    (at 43.18 27.94 180)
+    (at 38.1 20.32 270)
     (descr "Resistor, Axial_DIN0207 series, Axial, Horizontal, pin pitch=10.16mm, 0.25W = 1/4W, length*diameter=6.3*2.5mm^2, http://cdn-reichelt.de/documents/datenblatt/B400/1_4W%23YAG.pdf")
     (tags "Resistor Axial_DIN0207 series Axial Horizontal pin pitch 10.16mm 0.25W = 1/4W length 6.3mm diameter 2.5mm")
-    (fp_text reference R9 (at 5.08 2.37 180) (layer B.SilkS)
+    (fp_text reference R9 (at 5.08 2.37 270) (layer B.SilkS)
       (effects (font (size 1 1) (thickness 0.15)) (justify mirror))
     )
-    (fp_text value 10k (at 5.08 -2.37 180) (layer B.Fab)
+    (fp_text value 10k (at 5.08 -2.37 270) (layer B.Fab)
       (effects (font (size 1 1) (thickness 0.15)) (justify mirror))
     )
-    (fp_text user %R (at 5.08 0 180) (layer B.Fab)
+    (fp_text user %R (at 5.08 0 270) (layer B.Fab)
       (effects (font (size 1 1) (thickness 0.15)) (justify mirror))
     )
@@
     (fp_line (start 1.93 -1.25) (end 8.23 -1.25) (layer B.Fab) (width 0.1))
     (fp_line (start 1.93 1.25) (end 1.93 -1.25) (layer B.Fab) (width 0.1))
-    (pad 2 thru_hole oval (at 10.16 0 180) (size 1.6 1.6) (drill 0.8) (layers *.Cu *.Mask)
+    (pad 2 thru_hole oval (at 10.16 0 270) (size 1.6 1.6) (drill 0.8) (layers *.Cu *.Mask)
       (net 14 GND))
-    (pad 1 thru_hole circle (at 0 0 180) (size 1.6 1.6) (drill 0.8) (layers *.Cu *.Mask)
+    (pad 1 thru_hole circle (at 0 0 270) (size 1.6 1.6) (drill 0.8) (layers *.Cu *.Mask)
       (net 21 "Net-(Q3-Pad2)"))
     (model ${KISYS3DMOD}/Resistor_THT.3dshapes/R_Axial_DIN0207_L6.3mm_D2.5mm_P10.16mm_Horizontal.wrl
@@
   (gr_line (start 95.25 16.51) (end 95.25 46.99) (layer Edge.Cuts) (width 0.1))
   (gr_line (start 24.13 16.51) (end 95.25 16.51) (layer Edge.Cuts) (width 0.1))
-  (segment (start 27.94 35.56) (end 25.4 35.56) (width 2) (layer B.Cu) (net 24))
-  (segment (start 27.94 40.64) (end 25.4 40.64) (width 2) (layer B.Cu) (net 16))
   (segment (start 68.58 30.48) (end 73.66 30.48) (width 2) (layer B.Cu) (net 2))
   (segment (start 68.58 30.48) (end 66.04 30.48) (width 2) (layer B.Cu) (net 2))
@@
   (segment (start 88.9 22.86) (end 83.82 22.86) (width 2) (layer B.Cu) (net 14))
   (segment (start 83.82 22.86) (end 83.82 20.32) (width 2) (layer B.Cu) (net 14))
+  (segment (start 63.5 35.56) (end 66.04 35.56) (width 2) (layer B.Cu) (net 14))
+  (segment (start 27.94 40.64) (end 25.4 40.64) (width 2) (layer B.Cu) (net 16))
   (segment (start 40.64 43.18) (end 38.1 43.18) (width 2) (layer B.Cu) (net 16))
   (segment (start 40.64 38.1) (end 40.64 43.18) (width 2) (layer B.Cu) (net 16))
-  (segment (start 73.66 35.56) (end 76.2 35.56) (width 2) (layer B.Cu) (net 17))
   (segment (start 76.2 25.4) (end 73.66 25.4) (width 2) (layer B.Cu) (net 17))
-  (segment (start 76.2 35.56) (end 76.2 27.94) (width 2) (layer B.Cu) (net 17))
-  (segment (start 76.2 27.94) (end 86.36 27.94) (width 2) (layer B.Cu) (net 17))
-  (segment (start 76.2 27.94) (end 76.2 25.4) (width 2) (layer B.Cu) (net 17))
   (segment (start 86.36 27.94) (end 86.36 30.48) (width 2) (layer B.Cu) (net 17))
   (segment (start 86.36 30.48) (end 88.9 30.48) (width 2) (layer B.Cu) (net 17))
   (segment (start 63.5 43.18) (end 63.5 38.1) (width 2) (layer B.Cu) (net 17))
-  (segment (start 73.66 25.4) (end 71.12 25.4) (width 2) (layer B.Cu) (net 17))
   (segment (start 63.5 43.18) (end 66.04 43.18) (width 2) (layer B.Cu) (net 17))
   (segment (start 76.2 25.4) (end 78.74 25.4) (width 2) (layer B.Cu) (net 17))
@@
   (segment (start 73.66 20.32) (end 78.74 20.32) (width 2) (layer B.Cu) (net 17))
   (segment (start 78.74 20.32) (end 78.74 22.86) (width 2) (layer B.Cu) (net 17))
-  (segment (start 35.56 30.48) (end 38.1 30.48) (width 2) (layer B.Cu) (net 19))
-  (segment (start 38.1 30.48) (end 38.1 25.4) (width 2) (layer B.Cu) (net 19))
-  (segment (start 38.1 25.4) (end 40.64 25.4) (width 2) (layer B.Cu) (net 19))
+  (segment (start 78.74 35.56) (end 78.74 27.94) (width 2) (layer B.Cu) (net 17))
+  (segment (start 78.74 27.94) (end 86.36 27.94) (width 2) (layer B.Cu) (net 17))
+  (segment (start 73.66 35.56) (end 78.74 35.56) (width 2) (layer B.Cu) (net 17))
+  (segment (start 78.74 27.94) (end 78.74 25.4) (width 2) (layer B.Cu) (net 17))
   (segment (start 30.48 22.86) (end 33.02 22.86) (width 2) (layer B.Cu) (net 21))
   (segment (start 33.02 22.86) (end 33.02 20.32) (width 2) (layer B.Cu) (net 21))
   (segment (start 33.02 20.32) (end 35.56 20.32) (width 2) (layer B.Cu) (net 21))
+  (segment (start 35.56 20.32) (end 38.1 20.32) (width 2) (layer B.Cu) (net 21))
   (segment (start 68.58 22.86) (end 68.58 20.32) (width 2) (layer B.Cu) (net 23))
+  (segment (start 27.94 35.56) (end 25.4 35.56) (width 2) (layer B.Cu) (net 24))
   (segment (start 38.1 33.02) (end 40.64 33.02) (width 2) (layer B.Cu) (net 24))
 )

Commit message: Some schematic changes (dunno)
Parts:
- removed C1: 100nF, Capacitor_THT:C_Disc_D5.0mm_W2.5mm_P5.00mm
- removed Q1, Q2: 2N7000TA, Package_TO_SOT_THT:TO-92_Inline_Wide
- removed R2, R3, R4, R5: 10k, Resistor_THT:R_Axial_DIN0207_L6.3mm_D2.5mm_P10.16mm_Horizontal
- J3: value conn_display -> display_conn; footprint Connector_PinHeader_2.54mm:PinHeader_1x04_P2.54mm_Vertical -> Connector_PinHeader_2.54mm:PinHeader_1x08_P2.54mm_Vertical
- moved J3 23.4 mm to (71.1, 43.2), turned to 90 degrees
Connections:
- J3 pad 1: GND -> rst
- J3 pad 2: +5V -> GND
- J3 pad 3: sda_5v -> display_dc
- J3 pad 4: scl_5v -> display_din
- U1 pad 1: Net-(U1-Pad1) -> rst
Routing:
- net scl_5v: track 25.4 -> 2.54 mm
- net scl_3v: track 5.08 -> 0.00 mm
